File: TorqueSensorAmpifierPCB.kicad_sch (KiCad schematic)
At the start: 17 parts, among them J1 Conn_01x04_Socket, J2 Conn_01x04_Socket, U1 LM386

Commit message: Added Gerbers
Parts:
- added C2: .05uF, Capacitor_SMD:C_0805_2012Metric, symbol Device:C
- added R2: 10, Resistor_SMD:R_0805_2012Metric, symbol Device:R
- C2: value C -> 10uF
- C3: value C -> 250uF
- R1: footprint Resistor_SMD:R_0805_2012Metric -> Resistor_THT:R_Axial_DIN0614_L14.3mm_D5.7mm_P20.32mm_Horizontal
- R2: value R -> 1.2k
- U1: footprint Package_SO:SOIC-8-1EP_3.9x4.9mm_P1.27mm_EP2.41x3.3mm -> HCRL:M08A_TEX-L
Connections:
- net GND: now also C2.2
- net at C3.1, U1.5: now also R2.1
- new net: C2.1, R2.2
Other:
- moved on the sheet: C1, C2, C3, J1, J2, R2, TP1, TP2, TP3, TP4, U1

Commit message: Added BOMs
Parts:
- C1: value C -> 1uF; P/N (none) -> 0805B105K160NT
- C2: P/N (none) -> 0805X106K100CT
- R1: value R -> 5k; footprint Resistor_THT:R_Axial_DIN0614_L14.3mm_D5.7mm_P20.32mm_Horizontal -> Resistor_SMD:R_0805_2012Metric; P/N (none) -> ARG05BTC5001N
- R2: P/N (none) -> RS-05K122JT
- R2: P/N (none) -> CR0805F10R0P05Z
- U1: P/N (none) -> LM386MX-1/NOPB
Changed lines of the file:
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@@
   (symbol (lib_id "Device:C") (at 158.75 99.06 0) (unit 1)
     (in_bom yes) (on_board yes) (dnp no) (fields_autoplaced)
-    (property "Reference" "C1" (at 162.56 97.79 0)
-      (effects (font (size 1.27 1.27)) (justify left))
-    )
-    (property "Value" "C" (at 162.56 100.33 0)
+    (property "Reference" "C1" (at 162.56 98.425 0)
+      (effects (font (size 1.27 1.27)) (justify left))
+    )
+    (property "Value" "1uF" (at 162.56 100.965 0)
       (effects (font (size 1.27 1.27)) (justify left))
     )
@@
       (effects (font (size 1.27 1.27)) hide)
     )
+    (property "P/N" "0805B105K160NT" (at 158.75 99.06 0)
+      (effects (font (size 1.27 1.27)) hide)
+    )
     (pin "1")
     (pin "2")
@@
   (symbol (lib_id "Device:R") (at 90.17 86.36 0) (unit 1)
     (in_bom yes) (on_board yes) (dnp no) (fields_autoplaced)
-    (property "Reference" "R1" (at 92.075 85.09 0)
-      (effects (font (size 1.27 1.27)) (justify left))
-    )
-    (property "Value" "R" (at 92.075 87.63 0)
-      (effects (font (size 1.27 1.27)) (justify left))
-    )
-    (property "Footprint" "Resistor_THT:R_Axial_DIN0614_L14.3mm_D5.7mm_P20.32mm_Horizontal" (at 88.392 86.36 90)
+    (property "Reference" "R1" (at 92.71 85.725 0)
+      (effects (font (size 1.27 1.27)) (justify left))
+    )
+    (property "Value" "5k" (at 92.71 88.265 0)
+      (effects (font (size 1.27 1.27)) (justify left))
+    )
+    (property "Footprint" "Resistor_SMD:R_0805_2012Metric" (at 88.392 86.36 90)
       (effects (font (size 1.27 1.27)) hide)
     )
@@
       (effects (font (size 1.27 1.27)) hide)
     )
+    (property "P/N" "ARG05BTC5001N" (at 90.17 86.36 0)
+      (effects (font (size 1.27 1.27)) hide)
+    )
     (pin "1")
     (pin "2")
@@
       (effects (font (size 1.27 1.27)) hide)
     )
+    (property "P/N" "RS-05K122JT" (at 150.495 135.255 0)
+      (effects (font (size 1.27 1.27)) hide)
+    )
     (pin "1")
     (pin "2")
@@
     )
     (property "Datasheet" "~" (at 168.275 125.095 0)
+      (effects (font (size 1.27 1.27)) hide)
+    )
+    (property "P/N" "CR0805F10R0P05Z" (at 168.275 125.095 0)
       (effects (font (size 1.27 1.27)) hide)
     )
@@
       (effects (font (size 1.27 1.27)) hide)
     )
+    (property "P/N" "0805X106K100CT" (at 158.75 135.255 0)
+      (effects (font (size 1.27 1.27)) hide)
+    )
     (pin "1")
     (pin "2")
@@
       (effects (font (size 1.27 1.27)) hide)
     )
+    (property "P/N" "LM386MX-1/NOPB" (at 150.495 116.205 0)
+      (effects (font (size 1.27 1.27)) hide)
+    )
